File: ecad/transmission-lines/rf-switch/rf-switch.kicad_sch (KiCad schematic)
At the start: 5 parts, among them J1 USB_C_Receptacle_USB2.0, J2 Conn_01x05_Pin, SW1 SW_DIP_x01, U1 ADG918BRM, U2 AP7384-33Y

Commit message: rf-switch: Update
Parts:
- added C1: 10u, Capacitor_SMD:C_0603_1608Metric_Pad1.08x0.95mm_HandSolder, symbol Device:C
- added C2, C3: C, Capacitor_SMD:C_0603_1608Metric_Pad1.08x0.95mm_HandSolder, symbol Device:C
- added C4, C5: 100n, Capacitor_SMD:C_0603_1608Metric_Pad1.08x0.95mm_HandSolder, symbol Device:C
- added D1, D2: LED, LED_THT:LED_D3.0mm_FlatTop, symbol Device:LED
- added R1, R2: 1k, Resistor_SMD:R_0603_1608Metric_Pad0.98x0.95mm_HandSolder, symbol Device:R
- added R3, R4, R5, R8: R, Resistor_SMD:R_0603_1608Metric_Pad0.98x0.95mm_HandSolder, symbol Device:R
- added R6, R7: 56k, Resistor_SMD:R_0603_1608Metric_Pad0.98x0.95mm_HandSolder, symbol Device:R
- added U3: SN74LVC1G14DBV, Package_TO_SOT_SMD:SOT-23-5, symbol 74xGxx:SN74LVC1G14DBV
- SW1: footprint Button_Switch_SMD:SW_SPST_PTS645 -> Button_Switch_THT:SW_PUSH_6mm_H4.3mm
Connections:
- net at SW1.1: now also R2.2
- net at SW1.2: now also C1.1, R1.2, U3.2
- net +3.3V: now reaches U2.1 (VO)
- net +3.3V: now also U1.1 (VDD), C3.1, C4.1, C5.1, R1.1, R3.2, U3.5 (VCC)
- net GND: now reaches U2.2 (GND)
- net GND: now also J1.A1 (GND), J1.A12 (GND), J1.B1 (GND), J1.B12 (GND), J2.2 (Pin_2), J2.4 (Pin_4), U1.3 (GND), U1.6 (GND), U1.7 (GND), C1.2, C2.2, C3.2, C4.2, C5.2, D1.1 (K), D2.1 (K), R2.1, R5.1, R6.1, R7.1, U3.3 (GND)
- net VBUS: now reaches U2.3 (VI)
- net VBUS: now also J1.A4 (VBUS), J1.A9 (VBUS), J1.B4 (VBUS), J1.B9 (VBUS), C2.1
- net at J2.1 (Pin_1): now also U1.8 (RF1)
- net at J2.3 (Pin_3): now also U1.4 (RFC)
- net at J2.5 (Pin_5): now also U1.5 (RF2)
- net at J1.A5 (CC1): now also R7.2
- net at J1.A6 (D+): now also J1.B6 (D+), R8.1
- net at J1.A7 (D-): now also J1.B7 (D-), R8.2
- net at J1.B5 (CC2): now also R6.2
- net at J1.S1 (SHIELD): now also R5.2
- net Ctrl: now reaches U1.2 (CTRL)
- net Ctrl: now also R4.2, U3.4
- new net: D1.2 (A), R3.1
- new net: D2.2 (A), R4.1
- no-connect marks 0 -> 2
Other:
- moved on the sheet: J1, J2, SW1, U1, U2
